Commit message: Fix IMU configuration: Corrected serial port to /dev/rosmaster, enabled IMU publishing in driver, and uncommented imu_link in URDF

File: src/anzym_description/urdf/yahboomcar_X3plus.urdf.xacro (robot description, xacro)
@@ -8,5 +8,5 @@
     </material>
     <link name="base_footprint"/>
-    <!-- <link name="imu_link"/> -->
+    <link name="imu_link"/>
     <!-- common link-->
     <xacro:macro name="common_link" params="name material path *origin">
@@ -24,4 +24,7 @@
                 </geometry>
                 <origin xyz="0 0 0" rpy="0 0 0"/>
+                <collision>
+                    <origin xyz="0 0 0" rpy="0 0 0"/>
+                </collision>
             </collision>
             <xacro:insert_block name="origin"/>
@@ -81,5 +84,5 @@
         <origin xyz="0.0 0.0 0.076" rpy="0 0 0"/>
     </joint>
-    <!-- <xacro:fixed_joint name="base_imu" parent="base_link" child="imu_link" xyz="0.001 0.017 0.0322" rpy="0 3.1415 1.5707"/> -->
+    <xacro:fixed_joint name="base_imu" parent="base_link" child="imu_link" xyz="0.001 0.017 0.0322" rpy="0 3.1415 1.5707"/>
     <xacro:common_link name="laser_link" material="White" path="sensor">
         <inertial>
